File: Microcontroller Design/V1/V1.kicad_sch (KiCad schematic)
At the start: 50 parts, among them J1 U.FL-R-SMT_01_, J2 Conn_01x04, J3 USB_C_Receptacle, J4 Conn_01x02, SW1 SW_Push, U1 nRF9160-SIxA, U2 SIM-ST-MFF2, U3 SKY65404, U4 BQ25185DLHR, U5 CP2102N-Axx-xQFN20

Commit message: improved mc design
Parts:
- removed U3: SKY65404, RF:Skyworks_SKY65404-31, symbol RF_Amplifier:SKY65404
- added C22: 10nF, symbol Device:C
- added C23: 10uF, symbol Device:C
- added C24: 4.7uF, symbol Device:C
- added L1: 470nH, symbol Device:L
- added R15: 18k, symbol Device:R
- added R16: 162k, symbol Device:R
- added R7: 732k, symbol Device:R
- added TH1: 10k, symbol Device:Thermistor_NTC
- added U3: TLV73325PDBV, Package_TO_SOT_SMD:SOT-23-5, symbol Regulator_Linear:TLV73325PDBV
- added U6: MAX2679B, Package_BGA:WLP-4_0.83x0.83mm_P0.4mm, symbol RF_Amplifier:MAX2679B
- added U7: TPS62823DLC, Package_SON:Texas_VSON-HR-8_1.5x2mm_P0.5mm, symbol Regulator_Switching:TPS62823DLC
- C11: value 100nF -> 1000pF
- C12: value 10uF -> 10nF
- C8: value 100nF -> 0.1uF
Connections:
- net +3.3V: now also C24.2, L1.1, R7.1, U3.1 (IN); no longer C11.1, C12.1, C8.2, U4.1 (SYS)
- net GND: now also C8.2, U1.1 (GND_Shield), U1.103 (VSS), U1.11 (GND_Shield), U1.14 (GND_Shield), U1.17 (GND_Shield), U1.21 (GND_Shield), U1.27 (GND_Shield), U1.31 (GND_Shield), U1.36 (GND_Shield), U1.41 (GND_Shield), U1.44 (GND_Shield), U1.47 (GND_Shield), U1.5 (GND_Shield), U1.50 (GND_Shield), U1.52 (GND_Shield), U1.56 (GND_Shield), U1.6 (GND_Shield), U1.60 (GND_Shield), U1.62 (GND_Shield), U1.63 (GND_Shield), U1.65 (GND_Shield), U1.66 (GND_Shield), U1.68 (GND_Shield), U1.69 (GND_Shield), U1.7 (GND_Shield), U1.72 (GND_Shield), U1.74 (GND_Shield), U1.75 (GND_Shield), U1.76 (GND_Shield), U1.77 (GND_Shield), U1.78 (GND_Shield), U1.79 (GND_Shield), U1.8 (GND_Shield), U1.80 (GND_Shield), U1.81 (GND_Shield), U1.82 (GND_Shield), U1.85 (GND_Shield), U1.9 (GND_Shield), U1.90 (GND_Shield), U1.94 (GND_Shield), U1.98 (GND_Shield), C23.1, C24.1, R15.2, R16.1, TH1.2, U3.2 (GND), U6.B2 (G), U7.3 (AGND), U7.5 (PGND), U7.8 (PG); no longer C12.2
- net GPS: now also C12.1
- net LDO Killswitch: now reaches U1.4 (P0.07)
- net LDO Killswitch: now also U3.3 (EN)
- net NTC: now reaches U4.6 (TS/MR)
- net NTC: now also TH1.1
- net at U4.7 (ILIM/VSET): now also R15.1
- net at E1.1: now also C22.1
- new net: R16.2, R7.2, U7.2 (FB)
- new net: C22.2, U6.B1
- new net: C11.1, C8.1, U3.5 (OUT), U6.A1 (Vcc)
- new net: L1.2, U7.6 (SW)
- new net: C12.2, U6.A2
- new net SYS_OUT: C23.2, U4.1 (SYS), U7.1 (EN), U7.7 (VIN)
- no-connect marks 23 -> 51
Other:
- moved on the sheet: C10, C13, C14, C15, C16, C7, C9, D1, D2, D5, D6, E1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
